File: PCB/PCB.kicad_sch (KiCad schematic)
At the start: 0 parts

Commit message: boo
Parts:
- added C1, C10, C11, C12, C2, C3, C4, C5, C6, C7, C8, C9: 0.1uF, symbol Device:C_Small
- added R1, R2: 22, symbol Device:R_Small
- added R3: 10k, symbol Device:R_Small
- added SW1: RESET, symbol Switch:SW_Push
- added U1: RP2040, Package_DFN_QFN:QFN-56-1EP_7x7mm_P0.4mm_EP3.2x3.2mm, symbol MCU_RaspberryPi:RP2040
- added U2: W25Q32JVSS, Package_SO:SOIC-8_5.3x5.3mm_P1.27mm, symbol Memory_Flash:W25Q32JVSS
Connections:
- new net: C10.2, C11.2, C4.2, C5.2, C6.2, C7.2, C8.2, C9.2
- new net: R3.1, SW1.2, U1.26 (RUN)
- new net: R2.2, U1.46 (USB_DM)
- new net: R1.2, U1.47 (USB_DP)
- new net +1V1: C1.1, C2.1, C3.1, U1.23 (DVDD), U1.45 (VREG_VOUT), U1.50 (DVDD)
- new net +3V3: C10.1, C11.1, C12.1, C4.1, C5.1, C6.1, C7.1, C8.1, C9.1, R3.2, U1.1 (IOVDD), U1.10 (IOVDD), U1.22 (IOVDD), U1.33 (IOVDD), U1.42 (IOVDD), U1.43 (ADC_AVDD), U1.44 (VREG_IN), U1.48 (USB_VDD), U1.49 (IOVDD), U2.8 (VCC)
- new net DM: R2.1
- new net DP: R1.1
- new net GND: C1.2, C12.2, C2.2, C3.2, SW1.1, U1.19 (TESTEN), U1.57 (GND), U2.4 (GND)
- new net SPI_Q0: U1.53 (QSPI_SD0), U2.5 (DI/IO_{0})
- new net SPI_Q1: U1.55 (QSPI_SD1), U2.2 (DO/IO_{1})
- new net SPI_Q2: U1.54 (QSPI_SD2), U2.3 (~{WP}/IO_{2})
- new net SPI_Q3: U1.51 (QSPI_SD3), U2.7 (~{HOLD}/~{RESET}/IO_{3})
- new net SPI_SCLK: U1.52 (QSPI_SCLK), U2.6 (CLK)
- new net SPI_SS: U1.56 (QSPI_SS), U2.1 (~{CS})

Commit message: bleh v2
Parts:
- added J1: USB_C_Receptacle_USB2.0_16P, symbol Connector:USB_C_Receptacle_USB2.0_16P
- added R4, R6, R7: 10k, symbol Device:R_Small
- added R5: 1k, symbol Device:R_Small
- added SW2: Button, symbol Switch:SW_Push
Connections:
- net +3V3: now also J1.A4 (VBUS), J1.A9 (VBUS), J1.B4 (VBUS), J1.B9 (VBUS), R4.2
- net DM: now also J1.A7 (D-), J1.B7 (D-)
- net DP: now also J1.A6 (D+), J1.B6 (D+)
- net GND: now also C10.2, C11.2, C4.2, C5.2, C6.2, C7.2, C8.2, C9.2, J1.A1 (GND), J1.A12 (GND), J1.B1 (GND), J1.B12 (GND), J1.S1 (SHIELD), R6.2, R7.2, SW2.1
- net SPI_SS: now also R4.1, R5.1
- net XIN: now reaches U1.20 (XIN)
- net XOUT: now reaches U1.21 (XOUT)
- new net: J1.B5 (CC2), R7.1
- new net: J1.A5 (CC1), R6.1
- new net: R5.2, SW2.2

Commit message: this feels too easy. im scared
Parts:
- added C13, C14, C15, C16, C17, C18, C19, C20: 1uF, symbol Device:C_Small
- added C21, C23: 4.7uF, symbol Device:C_Small
- added D1, D2, D3: D_Small, symbol Device:D_Small
- added D4: LED, symbol Device:LED
- added L1: L_Small, symbol Device:L_Small
- added Q1: NMOS, symbol Simulation_SPICE:NMOS
- added R10, R8: 2.2, symbol Device:R_Small
- added R9: 1M, symbol Device:R_Small
- added U3: ~, symbol Taranium-libs:24_Pin_For_E_ink_display
- J1: footprint (none) -> Connector_USB:USB_C_Receptacle_HCTL_HC-TYPE-C-16P-01A
Connections:
- net +3V3: now also C21.2, L1.1, R10.2
- net GND: now also C13.2, C14.2, C15.2, C16.2, C17.2, C18.2, C19.2, C20.2, C21.1, D2.1 (K), D4.1 (K), R8.1, R9.1, U3.8 (BS1), U3.MP
- new net: C14.1, U3.15 (VDDIO), U3.16 (VCI)
- new net: C23.1, D3.2 (A), L1.2, Q1.1 (D)
- new net: C23.2, D1.1 (K), D2.2 (A)
- new net: C15.1, U3.18 (VDD)
- new net: D4.2 (A), R10.1
- new net: C19.1, U3.20 (VSH1)
- new net: C18.1, U3.22 (VSL)
- new net: C13.1, U3.5 (VSH2)
- new net BUSY: U3.9 (BUSY)
- new net CS: U3.12 (CS#)
- new net D/C: U3.11 (D/C#)
- new net GDR: Q1.2 (G), R9.2, U3.2 (GDR)
- new net RES: U3.10 (RES#)
- new net RESE: Q1.3 (S), R8.2, U3.3 (RESE)
- new net SCLK: U3.13 (SCL)
- new net SDI: U3.14 (SDA)
- new net VCOM: C16.1, U3.24 (VCOM)
- new net VGH: C20.1, D3.1 (K), U3.21 (VGH)
- new net VGL: C17.1, U3.23 (VGL)
Other:
- moved on the sheet: C1, C10, C11, C12, C2, C3, C4, C5, C6, C7, C8, C9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

Commit message: i am developing a hate of making footprints
Parts:
- C1, C10, C11, C12, C13, C14, C15, C16, C17, C18, C19, C2, C20, C21, C23, C3, C4, C5, C6, C7, C8, C9: footprint (none) -> Capacitor_SMD:C_01005_0402Metric
- D1, D2, D3: footprint (none) -> Diode_SMD:D_SOD-123
- D4: footprint (none) -> LED_SMD:LED_0805_2012Metric
- R1, R10, R2, R3, R4, R5, R6, R7, R8, R9: footprint (none) -> Resistor_SMD:R_01005_0402Metric
- SW1, SW2: footprint (none) -> Taranium-libs:C720477
Changed lines of the file:
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@@
 			)
 		)
-		(property "Footprint" ""
+		(property "Footprint" "Capacitor_SMD:C_01005_0402Metric"
 			(at 544.83 49.53 0)
 			(effects
@@
 			)
 		)
-		(property "Footprint" ""
+		(property "Footprint" "Capacitor_SMD:C_01005_0402Metric"
 			(at 340.36 231.14 0)
 			(effects
@@
 			)
 		)
-		(property "Footprint" ""
+		(property "Footprint" "Capacitor_SMD:C_01005_0402Metric"
 			(at 520.7 49.53 0)
 			(effects
@@
 			)
 		)
-		(property "Footprint" ""
+		(property "Footprint" "Capacitor_SMD:C_01005_0402Metric"
 			(at 332.74 248.92 0)
 			(effects
@@
 			)
 		)
-		(property "Footprint" ""
+		(property "Footprint" "Capacitor_SMD:C_01005_0402Metric"
 			(at 336.55 251.46 0)
 			(effects
@@
 			)
 		)
-		(property "Footprint" ""
+		(property "Footprint" "Capacitor_SMD:C_01005_0402Metric"
 			(at 387.35 232.41 0)
 			(effects
@@
 			)
 		)
-		(property "Footprint" ""
+		(property "Footprint" "Resistor_SMD:R_01005_0402Metric"
 			(at 528.32 168.91 0)
 			(effects
@@
 			)
 		)
-		(property "Footprint" ""
+		(property "Footprint" "Resistor_SMD:R_01005_0402Metric"
 			(at 347.98 59.69 0)
 			(effects
@@
 			)
 		)
-		(property "Footprint" ""
+		(property "Footprint" "Resistor_SMD:R_01005_0402Metric"
 			(at 425.45 80.01 0)
 			(effects
@@
 			)
 		)
-		(property "Footprint" ""
+		(property "Footprint" "Capacitor_SMD:C_01005_0402Metric"
 			(at 353.06 243.84 0)
 			(effects
@@
 			)
 		)
-		(property "Footprint" ""
+		(property "Footprint" "Resistor_SMD:R_01005_0402Metric"
 			(at 347.98 57.15 0)
 			(effects
@@
 			)
 		)
-		(property "Footprint" ""
+		(property "Footprint" "Capacitor_SMD:C_01005_0402Metric"
 			(at 335.28 236.22 0)
 			(effects
@@
 			)
 		)
-		(property "Footprint" ""
+		(property "Footprint" "Capacitor_SMD:C_01005_0402Metric"
 			(at 466.09 49.53 0)
 			(effects
@@
 			)
 		)
-		(property "Footprint" ""
+		(property "Footprint" "Diode_SMD:D_SOD-123"
 			(at 401.32 220.98 90)
 			(effects
@@
 			)
 		)
-		(property "Footprint" ""
+		(property "Footprint" "Capacitor_SMD:C_01005_0402Metric"
 			(at 433.07 49.53 0)
 			(effects
@@
 			)
 		)
-		(property "Footprint" ""
+		(property "Footprint" "Capacitor_SMD:C_01005_0402Metric"
 			(at 548.64 161.29 0)
 			(effects
@@
 			)
 		)
-		(property "Footprint" ""
+		(property "Footprint" "Capacitor_SMD:C_01005_0402Metric"
 			(at 477.52 49.53 0)
 			(effects
@@
 			)
 		)
-		(property "Footprint" ""
+		(property "Footprint" "Capacitor_SMD:C_01005_0402Metric"
 			(at 497.84 49.53 0)
 			(effects
@@
 			)
 		)
-		(property "Footprint" ""
+		(property "Footprint" "Capacitor_SMD:C_01005_0402Metric"
 			(at 533.4 49.53 0)
 			(effects
@@
 			)
 		)
-		(property "Footprint" ""
+		(property "Footprint" "Capacitor_SMD:C_01005_0402Metric"
 			(at 443.23 49.53 0)
 			(effects
@@
 			)
 		)
-		(property "Footprint" ""
+		(property "Footprint" "Resistor_SMD:R_01005_0402Metric"
 			(at 387.35 264.16 0)
 			(effects
@@
 			)
 		)
-		(property "Footprint" ""
+		(property "Footprint" "LED_SMD:LED_0805_2012Metric"
 			(at 368.3 137.16 0)
 			(effects
@@
 			)
 		)
-		(property "Footprint" ""
+		(property "Footprint" "Capacitor_SMD:C_01005_0402Metric"
 			(at 487.68 49.53 0)
 			(effects
@@
 			)
 		)
-		(property "Footprint" ""
+		(property "Footprint" "Capacitor_SMD:C_01005_0402Metric"
 			(at 368.3 247.65 0)
 			(effects
@@
 			)
 		)
-		(property "Footprint" ""
+		(property "Footprint" "Taranium-libs:C720477"
 			(at 513.08 166.37 0)
 			(effects
@@
 			)
 		)
-		(property "Footprint" ""
+		(property "Footprint" "Capacitor_SMD:C_01005_0402Metric"
 			(at 421.64 49.53 0)
 			(effects
@@
 			)
 		)
-		(property "Footprint" ""
+		(property "Footprint" "Resistor_SMD:R_01005_0402Metric"
 			(at 361.95 137.16 0)
 			(effects
@@
 			)
 		)
-		(property "Footprint" ""
+		(property "Footprint" "Resistor_SMD:R_01005_0402Metric"
 			(at 379.73 264.16 0)
 			(effects
@@
 			)
 		)
-		(property "Footprint" ""
+		(property "Footprint" "Capacitor_SMD:C_01005_0402Metric"
 			(at 346.71 241.3 0)
 			(effects
@@
 			)
 		)
-		(property "Footprint" ""
+		(property "Footprint" "Diode_SMD:D_SOD-123"
 			(at 397.51 242.57 90)
 			(effects
@@
 			)
 		)
-		(property "Footprint" ""
+		(property "Footprint" "Resistor_SMD:R_01005_0402Metric"
 			(at 427.99 93.98 0)
 			(effects
@@
 			)
 		)
-		(property "Footprint" ""
+		(property "Footprint" "Diode_SMD:D_SOD-123"
 			(at 401.32 231.14 90)
 			(effects
@@
 			)
 		)
-		(property "Footprint" ""
+		(property "Footprint" "Resistor_SMD:R_01005_0402Metric"
 			(at 427.99 91.44 0)
 			(effects
@@
 			)
 		)
-		(property "Footprint" ""
+		(property "Footprint" "Capacitor_SMD:C_01005_0402Metric"
 			(at 341.63 246.38 0)
 			(effects
@@
 			)
 		)
-		(property "Footprint" ""
+		(property "Footprint" "Capacitor_SMD:C_01005_0402Metric"
 			(at 509.27 49.53 0)
 			(effects
@@
 			)
 		)
-		(property "Footprint" ""
+		(property "Footprint" "Capacitor_SMD:C_01005_0402Metric"
 			(at 336.55 203.2 0)
 			(effects
@@
 			)
 		)
-		(property "Footprint" ""
+		(property "Footprint" "Taranium-libs:C720477"
 			(at 416.56 78.74 0)
 			(effects
@@
 			)
 		)
-		(property "Footprint" ""
+		(property "Footprint" "Resistor_SMD:R_01005_0402Metric"
 			(at 520.7 171.45 0)
 			(effects

Commit message: i feel like this footprint is wrong but its not idk
Parts:
- U3: footprint (none) -> Taranium-libs:05A20L24P
Changed lines of the file:
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@@
 			)
 		)
-		(property "Footprint" ""
+		(property "Footprint" "Taranium-libs:05A20L24P"
 			(at 313.69 220.98 0)
 			(effects

Commit message: everything is fine
Parts:
- U3: footprint Taranium-libs:05A20L24P -> Taranium-libs:FPC-SMD_24P-P0.50_05A20L24P
Changed lines of the file:
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@@
 		)
 	)
-	(global_label "BS"
-		(shape input)
-		(at 323.85 210.82 0)
-		(fields_autoplaced yes)
-		(effects
-			(font
-				(size 1.27 1.27)
-			)
-			(justify left)
-		)
-		(property "Intersheetrefs" "${INTERSHEET_REFS}"
-			(at 329.3147 210.82 0)
-			(effects
-				(font
-					(size 1.27 1.27)
-				)
-				(justify left)
-				(hide yes)
-			)
-		)
-	)
 	(global_label "SDI"
 		(shape input)
@@
 			)
 		)
-		(property "Footprint" "Taranium-libs:05A20L24P"
+		(property "Footprint" "Taranium-libs:FPC-SMD_24P-P0.50_05A20L24P"
 			(at 313.69 220.98 0)
 			(effects

Commit message: routing is fun
Parts:
- L1: footprint (none) -> Taranium-libs:IND-SMD_L6.0-W6.0_FNR60XXS
Changed lines of the file:
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@@
 			)
 		)
-		(property "Footprint" ""
+		(property "Footprint" "Taranium-libs:IND-SMD_L6.0-W6.0_FNR60XXS"
 			(at 375.92 242.57 0)
 			(effects

Commit message: amongus vias arent real, they cant hurt you. amongus vias:
Parts:
- added C22, C24: 10uF, Capacitor_SMD:C_01005_0402Metric, symbol Device:C_Small
- added C25, C26: 33pF, Capacitor_SMD:C_01005_0402Metric, symbol Device:C_Small
- added R11: 1k, Resistor_SMD:R_01005_0402Metric, symbol Device:R_Small
- added U4: NCP1117-3.3_SOT223, Package_TO_SOT_SMD:SOT-223-3_TabPin2, symbol Regulator_Linear:NCP1117-3.3_SOT223
- added Y1: 12 MHz, symbol Device:Crystal_GND24
- Q1: footprint (none) -> Package_TO_SOT_SMD:SOT-23
Connections:
- net +3V3: now also C24.1, U4.2 (VO); no longer J1.A4 (VBUS), J1.A9 (VBUS), J1.B4 (VBUS), J1.B9 (VBUS)
- net GND: now also C22.2, C24.2, C25.1, C26.1, U4.1 (GND), Y1.2, Y1.4
- net VGL: now also D1.2 (A)
- net XIN: now also C26.2, Y1.3
- net XOUT: now also R11.1
- new net: C25.2, R11.2, Y1.1
- new net VBUS: C22.1, J1.A4 (VBUS), J1.A9 (VBUS), J1.B4 (VBUS), J1.B9 (VBUS), U4.3 (VI)
Other:
- moved on the sheet: D4, R10
