File: PCB/PCB.kicad_sch (KiCad schematic)
At the start: 52 parts, among them J1 USB_C_Receptacle_USB2.0_14P, Q1 IRLML2060, SW1 SW_Push, SW2 SW_Push, U1 RP2040, U2 W25Q16JVSS, U4 NCP1117-3.3_SOT223, U5 USBLC6-2SC6, Y1 Crystal_GND24

Commit message: bleh
Parts:
- added C22, C28, C29: 1UF, Capacitor_SMD:C_0402_1005Metric, symbol Device:C_Small
- C21: value 1UF -> 100nf
- D2, D3, D4: value D_Small -> MBR0530
- L1: value L -> 10uh 1A
- R10: value 2.2 -> 0.47
- R11: value 1M -> 10k
- R6, R7: value 22 -> 90
- U4: value NCP1117-3.3_SOT223 -> XC6206P332MR; footprint Package_TO_SOT_SMD:SOT-223-3_TabPin2 -> Package_TO_SOT_SMD:SOT-23
Connections:
- net GND: now also U3.8 (BS1), C22.1, C28.1, C29.2
- net RESE: now also Q1.2 (S); no longer Q1.3 (D)
- net at C18.2, D4.2 (A), L1.1: now also Q1.3 (D); no longer Q1.2 (S)
- net at U3.19 (VPP): now also C29.1
- net at U3.4 (NC): now also C28.2
- net at U3.5 (VSH2): now also C22.2
- net BS: no longer names the net of U1.6 (GPIO4)
- net BS: no longer U3.8 (BS1)
- net DM renamed DN
Other:
- moved on the sheet: Q1

Commit message: push
Parts:
- U1: footprint Package_DFN_QFN:QFN-56-1EP_7x7mm_P0.4mm_EP3.2x3.2mm -> Package_DFN_QFN:QFN-56-1EP_7x7mm_P0.4mm_EP3.2x3.2mm_ThermalVias
Changed lines of the file:
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@@
 			)
 		)
-		(property "Footprint" "Package_DFN_QFN:QFN-56-1EP_7x7mm_P0.4mm_EP3.2x3.2mm"
+		(property "Footprint" "Package_DFN_QFN:QFN-56-1EP_7x7mm_P0.4mm_EP3.2x3.2mm_ThermalVias"
 			(at 350.52 78.74 0)
 			(effects

Commit message: commit
Parts:
- C10, C11, C12, C17, C2, C3, C4, C5, C6, C7, C8: value 0.1uf -> 100nf
- J1: value USB_C_Receptacle_USB2.0_14P -> C309365
- SW1, SW2: value SW_Push -> C720477
- Y1: value Crystal_GND24 -> C9002
Changed lines of the file:
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@@
 			)
 		)
-		(property "Value" "SW_Push"
+		(property "Value" "C720477"
 			(at 312.42 35.56 0)
 			(effects
@@
 			)
 		)
-		(property "Value" "0.1uf"
+		(property "Value" "100nf"
 			(at 402.59 21.5962 0)
 			(effects
@@
 			)
 		)
-		(property "Value" "USB_C_Receptacle_USB2.0_14P"
+		(property "Value" "C309365"
 			(at 33.02 34.29 0)
 			(effects
@@
 			)
 		)
-		(property "Value" "0.1uf"
+		(property "Value" "100nf"
 			(at 318.77 21.5962 0)
 			(effects
@@
 			)
 		)
-		(property "Value" "0.1uf"
+		(property "Value" "100nf"
 			(at 250.1963 22.86 90)
 			(effects
@@
 			)
 		)
-		(property "Value" "0.1uf"
+		(property "Value" "100nf"
 			(at 354.33 21.5962 0)
 			(effects
@@
 		(on_board yes)
 		(dnp no)
-		(fields_autoplaced yes)
 		(property "Reference" "Y1"
 			(at 213.36 82.6768 90)
@@
 			)
 		)
-		(property "Value" "Crystal_GND24"
-			(at 213.36 85.2168 90)
+		(property "Value" "C9002"
+			(at 201.676 81.788 90)
 			(effects
 				(font
@@
 			)
 		)
-		(property "Value" "0.1uf"
+		(property "Value" "100nf"
 			(at 363.22 21.5962 0)
 			(effects
@@
 			)
 		)
-		(property "Value" "0.1uf"
+		(property "Value" "100nf"
 			(at 309.88 21.5962 0)
 			(effects
@@
 			)
 		)
-		(property "Value" "0.1uf"
+		(property "Value" "100nf"
 			(at 387.35 21.5962 0)
 			(effects
@@
 			)
 		)
-		(property "Value" "0.1uf"
+		(property "Value" "100nf"
 			(at 345.44 21.5962 0)
 			(effects
@@
 			)
 		)
-		(property "Value" "0.1uf"
+		(property "Value" "100nf"
 			(at 370.84 21.5962 0)
 			(effects
@@
 			)
 		)
-		(property "Value" "0.1uf"
+		(property "Value" "100nf"
 			(at 396.24 21.5962 0)
 			(effects
@@
 			)
 		)
-		(property "Value" "0.1uf"
+		(property "Value" "100nf"
 			(at 117.602 40.386 90)
 			(effects
@@
 			)
 		)
-		(property "Value" "SW_Push"
+		(property "Value" "C720477"
 			(at 218.44 30.48 0)
 			(effects

Commit message: banana
Parts:
- U1: value RP2040 -> C2040
Changed lines of the file:
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@@
 			)
 		)
-		(property "Value" "RP2040"
+		(property "Value" "C2040"
 			(at 352.6633 125.73 0)
 			(effects

Commit message: journal 1
Parts:
- Q1: value IRLML2060 -> C5122027
Changed lines of the file:
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@@
 			)
 		)
-		(property "Value" "IRLML2060"
+		(property "Value" "C5122027"
 			(at 233.68 194.3101 0)
 			(effects

Commit message: bleh
Parts:
- D1: value LED -> C2293
Changed lines of the file:
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@@
 			)
 		)
-		(property "Value" "LED"
+		(property "Value" "C2293"
 			(at 251.1425 71.12 0)
 			(effects

Commit message: Cleanup Schematic
Parts:
- U3: value ~ -> (none)
Connections:
- net +5V: no longer C16.1, J1.A4 (VBUS), J1.A9 (VBUS), J1.B4 (VBUS), J1.B9 (VBUS), U4.3 (VI)
- new net VBUS: C16.1, J1.A4 (VBUS), J1.A9 (VBUS), J1.B4 (VBUS), J1.B9 (VBUS), U4.3 (VI)
Other:
- moved on the sheet: C1, C10, C11, C12, C13, C14, C17, C18, C19, C2, C20, C21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

Commit message: push
Parts:
- R6, R7: value 90 -> 22
Changed lines of the file:
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@@
 			)
 		)
-		(property "Value" "90"
+		(property "Value" "22"
 			(at 33.02 96.52 90)
 			(show_name no)
@@
 			)
 		)
-		(property "Value" "90"
+		(property "Value" "22"
 			(at 32.766 93.98 90)
 			(show_name no)
