File: PCB/PCB.kicad_pcb (KiCad board)
At the start: 2 copper layers, 100 x 63 mm, 52 parts, among them J1 USB_C_Receptacle_USB2.0_16P, Q1 NMOS, SW1 RESET, SW2 Button, U1 RP2040, U2 W25Q32JVSS, U4 NCP1117-3.3_SOT223, Y1 12 MHz

Commit message: COMMIT
Parts:
- SW2: value Button -> BOOT
- moved C21 0.74 mm to (121.1, 70.0)
Routing:
- net Net-(U1-RUN): track 40.5 -> 39.8 mm
Other:
- outline, holes or cut-outs redrawn

Commit message: bleh
Parts:
- moved C9 1.44 mm to (104.7, 83.3), turned to 45 degrees
- moved C8 0.97 mm to (103.9, 82.5), turned to 45 degrees
Routing:
- net BS: track 73.2 -> 71.3 mm
Changed lines of the file:
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@@
 	(footprint "Capacitor_SMD:C_0402_1005Metric"
 		(layer "F.Cu")
-		(at 104.7 83.12)
+		(at 103.94 82.51 45)
 		(descr "Capacitor SMD 0402 (1005 Metric), square (rectangular) end terminal, IPC-7351 nominal, (Body size source: IPC-SM-782 page 76, https://www.pcb-3d.com/wordpress/wp-content/uploads/ipc-sm-782a_amendment_1_and_2.pdf), generated with kicad-footprint-generator")
 		(tags "capacitor")
 		(property "Reference" "C8"
-			(at 0 -1.16 0)
+			(at -1.951615 -0.056569 45)
 			(layer "F.SilkS")
 			(effects
@@
 		)
 		(property "Value" "0.1uF"
-			(at 0 1.16 0)
+			(at 0 1.16 45)
 			(layer "F.Fab")
 			(effects
@@
 		)
 		(property "Datasheet" ""
-			(at 0 0 0)
+			(at 0 0 45)
 			(layer "F.Fab")
 			(hide yes)
@@
 		)
 		(property "Description" "Unpolarized capacitor, small symbol"
-			(at 0 0 0)
+			(at 0 0 45)
 			(layer "F.Fab")
 			(hide yes)
@@
 		)
 		(fp_text user "${REFERENCE}"
-			(at 0 0 0)
+			(at 0 0 45)
 			(layer "F.Fab")
 			(effects
@@
 		)
 		(pad "1" smd roundrect
-			(at -0.48 0)
+			(at -0.48 0 45)
 			(size 0.56 0.62)
 			(layers "F.Cu" "F.Mask" "F.Paste")
@@
 		)
 		(pad "2" smd roundrect
-			(at 0.48 0)
+			(at 0.48 0 45)
 			(size 0.56 0.62)
 			(layers "F.Cu" "F.Mask" "F.Paste")
@@
 	(footprint "Capacitor_SMD:C_0402_1005Metric"
 		(layer "F.Cu")
-		(at 105.8 84.3)
+		(at 104.729411 83.340589 45)
 		(descr "Capacitor SMD 0402 (1005 Metric), square (rectangular) end terminal, IPC-7351 nominal, (Body size source: IPC-SM-782 page 76, https://www.pcb-3d.com/wordpress/wp-content/uploads/ipc-sm-782a_amendment_1_and_2.pdf), generated with kicad-footprint-generator")
 		(tags "capacitor")
 		(property "Reference" "C9"
-			(at 2.3 -0.2 0)
+			(at -1.915426 0.148492 45)
 			(layer "F.SilkS")
 			(effects
@@
 		)
 		(property "Value" "0.1uF"
-			(at 0 1.16 0)
+			(at 0 1.16 45)
 			(layer "F.Fab")
 			(effects
@@
 		)
 		(property "Datasheet" ""
-			(at 0 0 0)
+			(at 0 0 45)
 			(layer "F.Fab")
 			(hide yes)
@@
 		)
 		(property "Description" "Unpolarized capacitor, small symbol"
-			(at 0 0 0)
+			(at 0 0 45)
 			(layer "F.Fab")
 			(hide yes)
@@
 		)
 		(fp_text user "${REFERENCE}"
-			(at 0 0 0)
+			(at 0 0 45)
 			(layer "F.Fab")
 			(effects
@@
 		)
 		(pad "1" smd roundrect
-			(at -0.48 0)
+			(at -0.48 0 45)
 			(size 0.56 0.62)
 			(layers "F.Cu" "F.Mask" "F.Paste")
@@
 		)
 		(pad "2" smd roundrect
-			(at 0.48 0)
+			(at 0.48 0 45)
 			(size 0.56 0.62)
 			(layers "F.Cu" "F.Mask" "F.Paste")
@@
 		)
 		(stroke
-			(width 0)
+			(width 0.1)
 			(type solid)
 		)
@@
 		)
 		(stroke
-			(width 0)
+			(width 0.1)
 			(type solid)
 		)
@@
 		)
 		(stroke
-			(width 0)
+			(width 0.1)
 			(type solid)
 		)
@@
 	)
 	(segment
-		(start 104.916176 83.82)
-		(end 104.916176 83.896176)
+		(start 106.3 71.9)
+		(end 106.3 72.968528)
 		(width 0.2)
 		(layer "F.Cu")
@@
 	)
 	(segment
-		(start 106.3 71.9)
-		(end 106.3 72.968528)
+		(start 92.6166 78.171)
+		(end 96.519012 78.171)
 		(width 0.2)
 		(layer "F.Cu")
@@
 	)
 	(segment
-		(start 105.15 84.57081)
-		(end 105.15 84.47)
+		(start 103.600589 82.890589)
+		(end 104.39 83.68)
 		(width 0.2)
 		(layer "F.Cu")
@@
 	)
 	(segment
-		(start 92.6166 78.171)
-		(end 96.519012 78.171)
+		(start 106.24 73.028528)
+		(end 106.24 73.1)
 		(width 0.2)
 		(layer "F.Cu")
@@
 	)
 	(segment
-		(start 106.24 73.028528)
-		(end 106.24 73.1)
+		(start 105.15 84.44)
+		(end 105.15 84.57081)
 		(width 0.2)
 		(layer "F.Cu")
@@
 	)
 	(segment
-		(start 105.15 84.47)
-		(end 105.32 84.3)
-		(width 0.2)
-		(layer "F.Cu")
-		(net 2)
-	)
-	(segment
-		(start 104.916176 83.82)
-		(end 104.449 83.352824)
+		(start 104.39 83.68)
+		(end 105.15 84.44)
 		(width 0.2)
 		(layer "F.Cu")
@@
 	)
 	(segment
-		(start 96.519012 78.171)
-		(end 97.462214 77.227798)
+		(start 103.083827 82.849411)
+		(end 102.323573 82.089157)
 		(width 0.2)
 		(layer "F.Cu")
@@
 	)
 	(segment
-		(start 98.985006 79.934994)
-		(end 98.877135 79.827123)
+		(start 103.600589 82.849411)
+		(end 103.083827 82.849411)
 		(width 0.2)
 		(layer "F.Cu")
@@
 	)
 	(segment
-		(start 103.354416 83.12)
-		(end 102.323573 82.089157)
+		(start 96.519012 78.171)
+		(end 97.462214 77.227798)
+		(width 0.2)
+		(layer "F.Cu")
+		(net 2)
+	)
+	(segment
+		(start 98.985006 79.934994)
+		(end 98.877135 79.827123)
 		(width 0.2)
 		(layer "F.Cu")
@@
 	)
 	(segment
-		(start 104.916176 83.896176)
-		(end 105.32 84.3)
-		(width 0.2)
-		(layer "F.Cu")
-		(net 2)
-	)
-	(segment
 		(start 103.354727 75.626395)
 		(end 103.642133 75.626395)
@@
 	)
 	(segment
-		(start 104.449 83.352824)
-		(end 104.449 83.12)
-		(width 0.2)
-		(layer "F.Cu")
-		(net 2)
-	)
-	(segment
 		(start 100.0125 94.0325)
 		(end 100.6 94.62)
@@
 	)
 	(segment
-		(start 104.45 83.12)
-		(end 103.354416 83.12)
+		(start 103.600589 82.849411)
+		(end 103.600589 82.890589)
 		(width 0.2)
 		(layer "F.Cu")
@@
 	)
 	(segment
-		(start 105.65 83.67)
-		(end 106.28 84.3)
+		(start 82.08 93)
+		(end 81.56 93.52)
 		(width 0.2)
 		(layer "F.Cu")
@@
 	)
 	(segment
-		(start 82.08 93)
-		(end 81.56 93.52)
+		(start 105.183824 83.12)
+		(end 104.95 83.12)
 		(width 0.2)
 		(layer "F.Cu")
@@
 	)
 	(segment
-		(start 104.95 83.12)
-		(end 104.95 81.9171)
-		(width 0.2)
-		(layer "F.Cu")
-		(net 71)
-	)
-	(segment
 		(start 142.05 77.57)
 		(end 146.49 77.57)
@@
 	)
 	(segment
-		(start 105.65 83.586176)
-		(end 105.65 83.67)
-		(width 0.2)
-		(layer "F.Cu")
-		(net 71)
-	)
-	(segment
 		(start 106.3 74.22)
 		(end 107.18 74.22)
@@
 	)
 	(segment
-		(start 104.95 81.9171)
-		(end 104.116283 81.083383)
+		(start 105.667644 83.6)
+		(end 105.068822 83.001178)
 		(width 0.2)
 		(layer "F.Cu")
@@
 	)
 	(segment
+		(start 104.95 82.841178)
+		(end 104.116283 82.007461)
+		(width 0.2)
+		(layer "F.Cu")
+		(net 71)
+	)
+	(segment
+		(start 104.116283 82.007461)
+		(end 104.116283 81.083383)
+		(width 0.2)
+		(layer "F.Cu")
+		(net 71)
+	)
+	(segment
+		(start 104.95 83.12)
+		(end 104.95 82.841178)
+		(width 0.2)
+		(layer "F.Cu")
+		(net 71)
+	)
+	(segment
 		(start 81.66 97.32)
 		(end 82.6 97.32)
@@
 	)
 	(segment
-		(start 104.95 83.12)
-		(end 105.183824 83.12)
-		(width 0.2)
-		(layer "F.Cu")
-		(net 71)
-	)
-	(segment
 		(start 111.5 75.55)
 		(end 111.9 75.55)
@@
 	)
 	(segment
-		(start 112.78 71.22)
-		(end 112.9 71.1)
+		(start 105.89 83.6)
+		(end 105.667644 83.6)
 		(width 0.2)
 		(layer "F.Cu")
@@
 	)
 	(segment
-		(start 144.8 67.92)
-		(end 144.9 67.82)
+		(start 112.78 71.22)
+		(end 112.9 71.1)
 		(width 0.2)
 		(layer "F.Cu")
@@
 	)
 	(segment
-		(start 106.7 84.3)
-		(end 107.3 84.9)
+		(start 144.8 67.92)
+		(end 144.9 67.82)
 		(width 0.2)
 		(layer "F.Cu")
@@
 	)
 	(segment
-		(start 106.28 84.3)
-		(end 106.7 84.3)
-		(width 0.2)
-		(layer "F.Cu")
-		(net 71)
-	)
-	(segment
 		(start 96.9 94.1)
 		(end 96.7 93.9)
@@
 	)
 	(segment
-		(start 105.183824 83.12)
-		(end 105.65 83.586176)
-		(width 0.2)
-		(layer "F.Cu")
-		(net 71)
-	)
-	(segment
 		(start 109.8 73.85)
 		(end 111.5 75.55)
@@
 	)
 	(via
-		(at 107.3 84.9)
+		(at 105.89 83.6)
 		(size 0.6)
 		(drill 0.3)

Commit message: blah bleh
Parts:
- moved C14 0.92 mm to (142.6, 74.1)
- moved C15 0.92 mm to (142.6, 72.6)
- moved C19 0.92 mm to (142.5, 71.4)
- moved C20 0.92 mm to (142.5, 70.3)
- moved C25 0.87 mm to (111.4, 72.0)
- moved C3 0.40 mm to (104.0, 73.0)
- moved C5 0.30 mm to (98.9, 74.1), turned to -135 degrees
Routing:
- net BS: track 71.3 -> 69.2 mm, vias 149 -> 148
- net Net-(U3-VDD): track 4.32 -> 3.35 mm
- net Net-(U3-VCI): track 4.81 -> 3.84 mm
- net VGH: track 11.5 -> 12.4 mm
- net Net-(U1-USB_DM): track 22.3 -> 23.3 mm
- net Net-(U3-VSH1): track 4.48 -> 3.79 mm

Commit message: update
Other:
- board text added: "BOOT"
Changed lines of the file:
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@@
 		(tags "resistor")
 		(property "Reference" "R10"
-			(at 0 -1.17 0)
+			(at 0 1.13 0)
 			(layer "F.SilkS")
 			(effects
@@
 	(gr_poly
 		(pts
-			(xy 84.089999 62.884999) (xy 58.690001 62.884999) (xy 58.690001 43.835001) (xy 84.089999 43.835001)
-		)
-		(stroke
-			(width 0.1)
-			(type solid)
-		)
-		(fill no)
-		(layer "F.Mask")
-	)
-	(gr_poly
-		(pts
-			(xy 171.344211 60.384689) (xy 145.944213 60.384689) (xy 145.944213 41.334691) (xy 171.344211 41.334691)
-		)
-		(stroke
-			(width 0.1)
-			(type solid)
-		)
-		(fill no)
-		(layer "F.Mask")
-	)
-	(gr_poly
-		(pts
 			(xy 76.619407 48.89077) (xy 76.649567 48.907811) (xy 76.678154 48.936114) (xy 76.705343 48.975023)
 			(xy 76.75622 49.082024) (xy 76.803588 49.22355) (xy 76.848836 49.394339) (xy 76.893356 49.589127)
@@
 	(gr_poly
 		(pts
-			(xy 161.37 57.99) (xy 151.210001 57.99) (xy 151.210001 50.370001) (xy 161.37 50.370001)
-		)
-		(stroke
-			(width 0.1)
-			(type solid)
-		)
-		(fill no)
-		(layer "F.Mask")
-	)
-	(gr_poly
-		(pts
 			(xy 80.787498 69.084377) (xy 105.989062 69.084377) (xy 105.989062 62.734377) (xy 80.787498 62.734377)
 		)
@@
 		)
 	)
+	(gr_text "BOOT"
+		(at 118.3 101.85 0)
+		(layer "F.SilkS")
+		(effects
+			(font
+				(size 1 1)
+				(thickness 0.1)
+			)
+		)
+	)
 	(segment
 		(start 97.2 82.634214)
@@
 	)
 	(group ""
-		(members "451b3c13-c63e-46a6-aab2-b49863a64c09" "a4636dba-bab8-4d83-b1a3-c9700dc98da8")
+		(members "a4636dba-bab8-4d83-b1a3-c9700dc98da8")
 	)
 	(group ""
-		(members "24d717db-1f11-4602-b0cb-e74afcce6b0c" "a2c6dc76-4de9-47da-8af9-f1bf16c847a0")
+		(members "a2c6dc76-4de9-47da-8af9-f1bf16c847a0")
 	)
 	(group ""
-		(members "2110b651-86d2-4cf3-a962-6edb4d9de154" "f2964559-d105-4b0c-8f9c-6e6138a3658d")
+		(members "2110b651-86d2-4cf3-a962-6edb4d9de154")
 	)
 	(group ""

Commit message: 83 error tags :D
Parts:
- J1: footprint Connector_USB:USB_C_Receptacle_HCTL_HC-TYPE-C-16P-01A -> Taranium-libs:USB-C-SMD_20P-P0.50-L6.5-W8.9
- moved C13 1.75 mm to (143.3, 79.0)
- moved R8 1.75 mm to (143.3, 80.0)
- moved J1 0.33 mm to (74.5, 95.2), turned to 0 degrees
Routing:
- net BS: track 69.2 -> 78.1 mm, vias 148 -> 159
- net VBUS: track 31.2 -> 35.7 mm
- net DM: track 7.25 -> 9.87 mm
- net Net-(U3-VSH2): track 4.66 -> 2.65 mm
- net Net-(J1-CC1): track 2.77 -> 3.92 mm
- net Net-(J1-CC2): track 2.90 -> 4.01 mm
- net DP: track 7.26 -> 8.22 mm
